Commit message: update

File: urdf/gen3_robotiq_2f_140_backup.urdf (robot description, URDF)
Before this commit: robot gen3_robotiq_2f_140, 24 links, 23 joints
Joints:
- joint joint_1: limit lower=-3.141592 upper=3.141592 effort=54 velocity=1.3963 -> effort=39 velocity=1.3963
- joint joint_2: limit lower=-2.41 upper=2.41 effort=54 velocity=1.3963 -> lower=-2.41 upper=2.41 effort=39 velocity=1.3963
- joint joint_3: limit lower=-3.141592 upper=3.141592 effort=54 velocity=1.3963 -> effort=39 velocity=1.3963
- joint joint_4: limit lower=-2.66 upper=2.66 effort=54 velocity=1.3963 -> lower=-2.66 upper=2.66 effort=39 velocity=1.3963
- joint joint_5: limit lower=-3.141592 upper=3.141592 effort=9 velocity=1.2218 -> effort=9 velocity=1.2218
- joint joint_7: limit lower=-3.141592 upper=3.141592 effort=9 velocity=1.2218 -> effort=9 velocity=1.2218

File: urdf/gen3_robotiq_2f_140_ver1.urdf (robot description, URDF)
Before this commit: robot gen3_robotiq_2f_140, 24 links, 23 joints
Joints:
- joint joint_1: limit lower=-3.141592 upper=3.141592 effort=54 velocity=1.3963 -> lower=-3.141592 upper=3.141592 effort=39 velocity=1.3963
- joint joint_2: limit lower=-2.41 upper=2.41 effort=54 velocity=1.3963 -> lower=-2.41 upper=2.41 effort=39 velocity=1.3963
- joint joint_3: limit lower=-3.141592 upper=3.141592 effort=54 velocity=1.3963 -> lower=-3.141592 upper=3.141592 effort=39 velocity=1.3963
- joint joint_4: limit lower=-2.66 upper=2.66 effort=54 velocity=1.3963 -> lower=-2.66 upper=2.66 effort=39 velocity=1.3963
